Commit message: Add robot demo into Gazebo

File: src/my_cutom_robot/description/robot.urdf.xacro (robot description, xacro)
@@ -2,3 +2,4 @@
 <robot xmlns:xacro="http://www.ros.org/wiki/xacro"  name="robot">
   <xacro:include filename="robot_core.xacro" />
+  <xacro:include filename="gazebo_control.xacro" />
 </robot>

File: src/my_cutom_robot/description/robot_core.xacro (robot description, xacro)
@@ -37,4 +37,8 @@
         </xacro:inertial_box>
     </link>
+    <!-- Add color into gazebo by adding gazebo tag -->
+    <gazebo reference="chassis">
+        <material>Gazebo/White</material>
+    </gazebo>
     <!-- Left wheel -->
     <joint name="left_wheel_joint" type="continuous">
@@ -61,6 +65,9 @@
         </xacro:inertial_cylinder>
     </link>
+    <gazebo reference="left_wheel">
+        <material>Gazebo/Blue</material>
+    </gazebo>
     <!-- Right wheel -->
-    <joint name="rigth_wheel_joint" type="continuous">
+    <joint name="right_wheel_joint" type="continuous">
         <parent link="base_link" />
         <child link="right_wheel" />
@@ -85,4 +92,7 @@
         </xacro:inertial_cylinder>
     </link>
+    <gazebo reference="right_wheel">
+        <material>Gazebo/Blue</material>
+    </gazebo>
     <joint name="caster_wheel_joint" type="fixed">
         <parent link="chassis" />
@@ -107,3 +117,8 @@
         </xacro:inertial_sphere>
     </link>
+    <gazebo reference="caster_wheel">
+        <material>Gazebo/Black</material>
+        <mu1 value="0.001" />
+        <mu2 value="0.001" />
+    </gazebo>
 </robot>
