Commit message: Add a camera

File: src/my_cutom_robot/description/lidar.xacro (robot description, xacro)
@@ -9,21 +9,21 @@
         <visual>
             <geometry>
-                <cylinder radius="0.05" length="0.04" />
+                <cylinder radius="0.05" length="0.04"/>
             </geometry>
-            <material name="blue" />
+            <material name="red"/>
         </visual>
         <collision>
             <geometry>
-              <cylinder radius="0.05" length="0.04" />
+                <cylinder radius="0.05" length="0.04"/>
             </geometry>
         </collision>
         <xacro:inertial_cylinder mass="0.1" length="0.04" radius="0.05">
-            <origin xyz="0 0 0" rpy="0 0 0" />
+            <origin xyz="0 0 0" rpy="0 0 0"/>
         </xacro:inertial_cylinder>
     </link>
-    <!-- To add a lidar frame into Gazebo, tags below maybe a bit of complicated -->
     <gazebo reference="laser_frame">
+        <material>Gazebo/Red</material>
         <sensor name="laser" type="ray">
-            <pose>0 0 0 0 0 0</pose>
+            <pose> 0 0 0 0 0 0 </pose>
             <visualize>true</visualize>
             <update_rate>10</update_rate>
@@ -32,5 +32,4 @@
                     <horizontal>
                         <samples>360</samples>
-                        <resolution>1</resolution>
                         <min_angle>-3.14</min_angle>
                         <max_angle>3.14</max_angle>
@@ -40,14 +39,10 @@
                     <min>0.3</min>
                     <max>12</max>
-                    <resolution>0.01</resolution>
                 </range>
-                <plugin name="laser_controller" filename="libgazebo_ros_ray_sensor.so">
-                    <ros>
-                        <argument>~/out:=scan</argument>
-                    </ros>
-                    <output_type>sensoe_msgs/LaserScan</output_type>
-                    <frame_name>laser_frame</frame_name>
-                </plugin>
             </ray>
+            <plugin name="laser_controller" filename="libgazebo_ros_ray_sensor.so">
+                <output_type>sensor_msgs/LaserScan</output_type>
+                <frame_name>laser_frame</frame_name>
+            </plugin>
         </sensor>
     </gazebo>

File: src/my_cutom_robot/description/robot_core.xacro (robot description, xacro)
@@ -13,4 +13,7 @@
     <material name="black">
         <color rgba="0 0 0 1" />
+    </material>
+    <material name="red">
+        <color rgba="1 0 0 " />
     </material>
     <link name="base_link"></link>
